File: KiCad/Leafony_Template/Leafony_Template.kicad_sch (KiCad schematic)
At the start: 1 part, among them CN1 Leafony bus

Commit message: Update KiCad Template
Parts:
- removed CN1: Leafony bus, Leafony:CN_F29_B29, symbol Leafony:LeafIF
- added CN1: Leafony Bus, Leafony:CN_F29_B29, symbol Leafony:Leafony Bus
Connections:
- net A0: now also CN1.B6 (A0), CN1.F6 (A0)
- net A1: now also CN1.B8 (A1), CN1.F8 (A1)
- net A2: now also CN1.B10 (A2), CN1.F10 (A2)
- net A3: now also CN1.B12 (A3), CN1.F12 (A3)
- net A4: now also CN1.B14 (A4), CN1.F14 (A4)
- net A5: now also CN1.B16 (A5), CN1.F16 (A5)
- net AREF: now also CN1.B4 (AREF), CN1.F4 (AREF)
- net D0: now also CN1.B18 (D0), CN1.F18 (D0)
- net D1: now also CN1.B20 (D1), CN1.F20 (D1)
- net D10: now also CN1.B15 (D10), CN1.F15 (D10)
- net D11: now also CN1.B17 (D11), CN1.F17 (D11)
- net D12: now also CN1.B19 (D12), CN1.F19 (D12)
- net D13: now also CN1.B21 (D13), CN1.F21 (D13)
- net D2: now also CN1.B22 (D2), CN1.F22 (D2)
- net D3: now also CN1.B24 (D3), CN1.F24 (D3)
- net D4: now also CN1.B26 (D4), CN1.F26 (D4)
- net D5: now also CN1.B28 (D5), CN1.F28 (D5)
- net D6: now also CN1.B7 (D6), CN1.F7 (D6)
- net D7: now also CN1.B9 (D7), CN1.F9 (D7)
- net D8: now also CN1.B11 (D8), CN1.F11 (D8)
- net D9: now also CN1.B13 (D9), CN1.F13 (D9)
- net GND: now also CN1.B27 (GND), CN1.F27 (GND)
- net RESET: now also CN1.B5 (RESET), CN1.F5 (RESET)
- net SCL: now also CN1.B25 (SCL), CN1.F25 (SCL)
- net SDA: now also CN1.B23 (SDA), CN1.F23 (SDA)
- net SWCLK: now also CN1.B29 (SWCLK), CN1.F29 (SWCLK)
- net SWDIO: now also CN1.B2 (SWDIO), CN1.F2 (SWDIO)
- net VBUS: now also CN1.B3 (VBUS), CN1.F3 (VBUS)
- new net +3V3: CN1.B1 (3.3V), CN1.F1 (3.3V)
